Commit message: Implementando o controle usando o ROS Control

File: urdf/ackermann_robot.xacro (robot description, xacro)
@@ -150,36 +150,98 @@
   <joint name="front_left_steering_joint" type="revolute">
     <parent link="base_link"/>
-    <child link="steering_left_wheel"/>
+    <child link="front_left_steering_rotation_link"/>
     <origin xyz="0.2 0.2 0.1" rpy="0 0 0"/>
     <axis xyz="0 0 1"/>
     <limit lower="-0.5236" upper="0.5236" effort="10" velocity="1.0"/> <!-- Limite de direção (±30 graus) -->
   </joint>
+  <!--Link intermediário para a rotação da roda dianteira esquerda-->
+  <link name="front_left_steering_rotation_link">
+    <visual>
+        <geometry>
+            <box size="0.01 0.01 0.01"/>
+        </geometry>
+    </visual>
+    <inertial>
+        <mass value="0.01"/>
+        <inertia ixx="0.00001" ixy="0.0" ixz="0.0" iyy="0.00001" iyz="0.0" izz="0.00001"/>
+    </inertial>
+  </link>
+  <!-- Junta de rotação para o eixo y (rotação da roda) -->
+  <joint name="front_left_wheel_rotation_joint" type="continuous">
+      <parent link="front_left_steering_rotation_link"/>
+      <child link="steering_left_wheel"/>
+      <origin xyz="0 0 0" rpy="0 0 0"/>
+      <axis xyz="0 1 0"/>
+      <limit lower="0" upper="0" effort="50" velocity="10.0"/>
+  </joint>
   <joint name="front_right_steering_joint" type="revolute">
     <parent link="base_link"/>
-    <child link="steering_right_wheel"/>
+    <child link="front_right_steering_rotation_link"/>
     <origin xyz="0.2 -0.2 0.1" rpy="0 0 0"/>
     <axis xyz="0 0 1"/>
     <limit lower="-0.5236" upper="0.5236" effort="10" velocity="1.0"/> <!-- Limite de direção (±30 graus) -->
   </joint>
-  <!-- Plugin para Ackermann Steering Control diretamente no Xacro -->
+  <!--Link intermediário para a rotação da roda dianteira esquerda-->
+  <link name="front_right_steering_rotation_link">
+    <visual>
+        <geometry>
+            <box size="0.01 0.01 0.01"/>
+        </geometry>
+    </visual>
+    <inertial>
+        <mass value="0.01"/>
+        <inertia ixx="0.00001" ixy="0.0" ixz="0.0" iyy="0.00001" iyz="0.0" izz="0.00001"/>
+    </inertial>
+  </link>
+  <!-- Junta de rotação para o eixo y (rotação da roda) -->
+  <joint name="front_right_wheel_rotation_joint" type="continuous">
+    <parent link="front_right_steering_rotation_link"/>
+    <child link="steering_right_wheel"/>
+    <origin xyz="0 0 0" rpy="0 0 0"/>
+    <axis xyz="0 1 0"/>
+    <limit effort="100" velocity="100"/>
+    <joint_properties damping="1.0" friction="1.0"/>
+  </joint>
+<transmission name="front_left_steering_trans">
+  <type>transmission_interface/SimpleTransmission</type>
+  <joint name="front_left_steering_joint">
+    <hardwareInterface>hardware_interface/EffortJointInterface</hardwareInterface>
+  </joint>
+  <actuator name="front_left_steering_motor">
+    <mechanicalReduction>1</mechanicalReduction>
+  </actuator>
+</transmission>
+<transmission name="front_right_steering_trans">
+  <type>transmission_interface/SimpleTransmission</type>
+  <joint name="front_right_steering_joint">
+    <hardwareInterface>hardware_interface/EffortJointInterface</hardwareInterface>
+  </joint>
+  <actuator name="front_right_steering_motor">
+    <mechanicalReduction>1</mechanicalReduction>
+  </actuator>
+</transmission>
+<transmission name="rear_left_wheel_trans">
+  <type>transmission_interface/SimpleTransmission</type>
+  <joint name="rear_left_wheel_joint">
+    <!--hardwareInterface>hardware_interface/EffortJointInterface</hardwareInterface-->
+    <hardwareInterface>hardware_interface/VelocityJointInterface</hardwareInterface>
+  </joint>
+  <actuator name="rear_left_wheel_motor">
+    <mechanicalReduction>1</mechanicalReduction>
+  </actuator>
+</transmission>
+<transmission name="rear_right_wheel_trans">
+  <type>transmission_interface/SimpleTransmission</type>
+  <joint name="rear_right_wheel_joint">
+    <!--hardwareInterface>hardware_interface/EffortJointInterface</hardwareInterface-->
+    <hardwareInterface>hardware_interface/VelocityJointInterface</hardwareInterface>
+  </joint>
+  <actuator name="rear_right_wheel_motor">
+    <mechanicalReduction>1</mechanicalReduction>
+  </actuator>
+</transmission>
   <gazebo>
-    <plugin name="ackermann_steering_controller" filename="libackermann_steering_controller.so">
+    <plugin name="gazebo_ros_control" filename="libgazebo_ros_control.so">
       <robotNamespace>/</robotNamespace>
-      <rear_wheels>                   <!-- Juntas das rodas traseiras -->
-        rear_left_wheel_joint
-        rear_right_wheel_joint
-      </rear_wheels>
-      <front_steering>                <!-- Juntas de direção dianteiras -->
-        front_left_steering_joint
-        front_right_steering_joint
-      </front_steering>
-      <wheel_base>1.0</wheel_base>               <!-- Distância entre eixos -->
-      <wheel_radius>0.2</wheel_radius>           <!-- Raio das rodas -->
-      <steering_limit>0.5235987756</steering_limit> <!-- Limite de direção (±30 graus) -->
-      <cmd_vel_timeout>0.5</cmd_vel_timeout>     <!-- Tempo limite para comando no /cmd_vel -->
-      <base_frame_id>base_link</base_frame_id>   <!-- Frame base do robô -->
-      <enable_odom_tf>true</enable_odom_tf>      <!-- Publicar transformações de odometria -->
-      <publish_rate>50</publish_rate>            <!-- Taxa de publicação de odometria -->
-      <velocity_rolling_window_size>10</velocity_rolling_window_size> <!-- Janela de suavização de odometria -->
     </plugin>
   </gazebo>

Commit message: Acionando os sensores e alterando o nome de algumas variáveis

File: urdf/ackermann_robot.xacro (robot description, xacro)
@@ -3,4 +3,6 @@
   <xacro:property name="pi" value="3.14"/>
   <xacro:property name="wheel_roll_angle" value="${pi/2}"/>
+  <!--This link it is just to avoid a warning-->
+  <link name="dummy_link"/>
   <!-- Base Link (Chassis) -->
   <link name="base_link">
@@ -23,4 +25,10 @@
     </inertial>
   </link>
+  <!--This joint it is just to avoid a warning-->
+  <joint name="fixed_joint" type="fixed">
+    <parent link="dummy_link"/>
+    <child link="base_link"/>
+    <origin xyz="0 0 0" rpy="0 0 0"/>
+  </joint>
   <link name="steering_left_wheel">
     <visual>
@@ -148,7 +156,7 @@
   </joint>
     <!-- Juntas dianteiras (direcionadas) -->
-  <joint name="front_left_steering_joint" type="revolute">
+  <joint name="front_left_wheel_steering_joint" type="revolute">
     <parent link="base_link"/>
-    <child link="front_left_steering_rotation_link"/>
+    <child link="front_left_wheel_steering_rotation_link"/>
     <origin xyz="0.2 0.2 0.1" rpy="0 0 0"/>
     <axis xyz="0 0 1"/>
@@ -156,5 +164,5 @@
   </joint>
   <!--Link intermediário para a rotação da roda dianteira esquerda-->
-  <link name="front_left_steering_rotation_link">
+  <link name="front_left_wheel_steering_rotation_link">
     <visual>
         <geometry>
@@ -169,5 +177,5 @@
   <!-- Junta de rotação para o eixo y (rotação da roda) -->
   <joint name="front_left_wheel_rotation_joint" type="continuous">
-      <parent link="front_left_steering_rotation_link"/>
+      <parent link="front_left_wheel_steering_rotation_link"/>
       <child link="steering_left_wheel"/>
       <origin xyz="0 0 0" rpy="0 0 0"/>
@@ -175,7 +183,7 @@
       <limit lower="0" upper="0" effort="50" velocity="10.0"/>
   </joint>
-  <joint name="front_right_steering_joint" type="revolute">
+  <joint name="front_right_wheel_steering_joint" type="revolute">
     <parent link="base_link"/>
-    <child link="front_right_steering_rotation_link"/>
+    <child link="front_right_wheel_steering_rotation_link"/>
     <origin xyz="0.2 -0.2 0.1" rpy="0 0 0"/>
     <axis xyz="0 0 1"/>
@@ -183,5 +191,5 @@
   </joint>
   <!--Link intermediário para a rotação da roda dianteira esquerda-->
-  <link name="front_right_steering_rotation_link">
+  <link name="front_right_wheel_steering_rotation_link">
     <visual>
         <geometry>
@@ -196,5 +204,5 @@
   <!-- Junta de rotação para o eixo y (rotação da roda) -->
   <joint name="front_right_wheel_rotation_joint" type="continuous">
-    <parent link="front_right_steering_rotation_link"/>
+    <parent link="front_right_wheel_steering_rotation_link"/>
     <child link="steering_right_wheel"/>
     <origin xyz="0 0 0" rpy="0 0 0"/>
@@ -203,19 +211,19 @@
     <joint_properties damping="1.0" friction="1.0"/>
   </joint>
-<transmission name="front_left_steering_trans">
+<transmission name="front_left_wheel_steering_trans">
   <type>transmission_interface/SimpleTransmission</type>
-  <joint name="front_left_steering_joint">
+  <joint name="front_left_wheel_steering_joint">
     <hardwareInterface>hardware_interface/EffortJointInterface</hardwareInterface>
   </joint>
-  <actuator name="front_left_steering_motor">
+  <actuator name="front_left_wheel_steering_motor">
     <mechanicalReduction>1</mechanicalReduction>
   </actuator>
 </transmission>
-<transmission name="front_right_steering_trans">
+<transmission name="front_right_wheel_steering_trans">
   <type>transmission_interface/SimpleTransmission</type>
-  <joint name="front_right_steering_joint">
+  <joint name="front_right_wheel_steering_joint">
     <hardwareInterface>hardware_interface/EffortJointInterface</hardwareInterface>
   </joint>
-  <actuator name="front_right_steering_motor">
+  <actuator name="front_right_wheel_steering_motor">
     <mechanicalReduction>1</mechanicalReduction>
   </actuator>
@@ -241,4 +249,117 @@
   </actuator>
 </transmission>
+    <!-- IMU Sensor -->
+    <link name="imu_link">
+        <inertial>
+            <origin xyz="0 0 0" />
+            <mass value="0.01" />
+            <inertia ixx="0.0001" ixy="0" ixz="0" iyy="0.0001" iyz="0" izz="0.0001" />
+        </inertial>
+        <visual>
+            <origin xyz="0 0 0" />
+            <geometry>
+                <box size="0.01 0.01 0.01" />
+            </geometry>
+        </visual>
+    </link>
+    <joint name="imu_joint" type="fixed">
+        <parent link="base_link" />
+        <child link="imu_link" />
+        <origin xyz="0 0 0.16" rpy="0 0 0" />
+    </joint>
+    <gazebo reference="imu_link">
+        <sensor name="my_imu" type="imu">
+            <always_on>true</always_on>
+            <plugin name="my_imu_plugin" filename="libgazebo_ros_imu_sensor.so">
+                <topicName>/imu</topicName>
+                <updateRateHZ>100</updateRateHZ>
+                <frameName>imu_link</frameName>
+            </plugin>
+        </sensor>
+    </gazebo>
+    <!--Sensor LiDAR 2D -->
+    <link name="lidar_link">
+      <inertial>
+          <origin xyz="0 0 0" />
+          <mass value="0.01" />
+          <inertia ixx="0.0001" ixy="0" ixz="0" iyy="0.0001" iyz="0" izz="0.0001" />
+      </inertial>
+      <visual>
+          <origin xyz="0 0 0" />
+          <geometry>
+              <box size="0.01 0.01 0.01" />
+          </geometry>
+      </visual>
+    </link>
+    <joint name="lidar_joint" type="fixed">
+        <parent link="base_link" />
+        <child link="lidar_link" />
+        <origin xyz="0 0 0.21" rpy="0 0 0" />
+    </joint>
+    <gazebo reference="lidar_link">
+        <sensor type="ray" name="lidar_sensor">
+            <pose>0 0 0 0 0 0</pose>
+            <ray>
+                <scan>
+                    <horizontal>
+                        <samples>640</samples>
+                        <resolution>1</resolution>
+                        <min_angle>-${pi}</min_angle>
+                        <max_angle>${pi}</max_angle>
+                    </horizontal>
+                </scan>
+                <range>
+                    <min>0.08</min>
+                    <max>10</max>
+                    <resolution>0.01</resolution>
+                </range>
+                <noise>
+                    <type>gaussian</type>
+                    <mean>0.0</mean>
+                    <stddev>0.01</stddev>
+                </noise>
+            </ray>
+            <plugin name="gazebo_ros_laser" filename="libgazebo_ros_laser.so">
+                <!-- Publicar a nuvem de pontos no tópico /lidar/points -->
+                <topicName>/lidar/points</topicName>
+                <frameName>lidar_link</frameName>
+            </plugin>
+            <always_on>1</always_on>
+            <update_rate>30</update_rate>
+            <visualize>true</visualize>
+        </sensor>
+    </gazebo>
+  <!-- GPS Sensor -->
+  <link name="gps_link">
+    <inertial>
+        <origin xyz="0 0 0" />
+        <mass value="0.01" />
+        <inertia ixx="0.0001" ixy="0" ixz="0" iyy="0.0001" iyz="0" izz="0.0001" />
+    </inertial>
+    <visual>
+        <origin xyz="0 0 0" />
+        <geometry>
+            <box size="0.01 0.01 0.01" />
+        </geometry>
+    </visual>
+  </link>
+  <joint name="gps_joint" type="fixed">
+      <parent link="base_link" />
+      <child link="gps_link" />
+      <origin xyz="0 0 0.17" rpy="0 0 0" />
+  </joint>
+  <gazebo>
+    <plugin name="gps" filename="libhector_gazebo_ros_gps.so">
+      <alwaysOn>1</alwaysOn>
+      <updateRate>10.0</updateRate>
+      <bodyName>dummy_link</bodyName>
+      <topicName>fix</topicName>
+      <velocityTopicName>fix_velocity</velocityTopicName>
+      <drift>5.0 5.0 5.0</drift>
+      <gaussianNoise>0.1 0.1 0.1</gaussianNoise>
+      <velocityDrift>0 0 0</velocityDrift>
+      <velocityGaussianNoise>0.1 0.1 0.1</velocityGaussianNoise>
+    </plugin>
+   </gazebo>
   <gazebo>
     <plugin name="gazebo_ros_control" filename="libgazebo_ros_control.so">

Commit message: Adicionando as modificações para funcionar com o ackermann_steering_controller

File: urdf/ackermann_robot.xacro (robot description, xacro)
@@ -139,6 +139,17 @@
     </inertial>
   </link>
+  <!--Virtual link for steering-->
+  <link name="steering_link"/>
+  <!--Virtual link for the rear wheels -->
+  <link name="rear_axle_link">
+    <collision>
+      <origin xyz="0 0 0" rpy="0 0 0"/>
+      <geometry>
+        <cylinder radius="0.001" length="0.001"/>
+      </geometry>
+    </collision>
+  </link>
   <joint name="rear_left_wheel_joint" type="continuous">
-    <parent link="base_link"/>
+    <parent link="rear_axle_link"/>
     <child link="rear_left_wheel"/>
     <origin xyz="-0.2 0.2 0.1" rpy="0 0 0"/>
@@ -148,5 +159,5 @@
   </joint>
   <joint name="rear_right_wheel_joint" type="continuous">
-    <parent link="base_link"/>
+    <parent link="rear_axle_link"/>
     <child link="rear_right_wheel"/>
     <origin xyz="-0.2 -0.2 0.1" rpy="0 0 0"/>
@@ -155,13 +166,12 @@
     <joint_properties damping="1.0" friction="1.0"/>
   </joint>
-    <!-- Juntas dianteiras (direcionadas) -->
   <joint name="front_left_wheel_steering_joint" type="revolute">
-    <parent link="base_link"/>
+    <parent link="steering_link"/>
     <child link="front_left_wheel_steering_rotation_link"/>
     <origin xyz="0.2 0.2 0.1" rpy="0 0 0"/>
     <axis xyz="0 0 1"/>
-    <limit lower="-0.5236" upper="0.5236" effort="10" velocity="1.0"/> <!-- Limite de direção (±30 graus) -->
-  </joint>
-  <!--Link intermediário para a rotação da roda dianteira esquerda-->
+    <limit lower="-0.5236" upper="0.5236" effort="10" velocity="1.0"/> <!-- (±30 degrees) -->
+  </joint>
+  <!--Link to connect the steering and rotation joints-->
   <link name="front_left_wheel_steering_rotation_link">
     <visual>
@@ -175,5 +185,4 @@
     </inertial>
   </link>
-  <!-- Junta de rotação para o eixo y (rotação da roda) -->
   <joint name="front_left_wheel_rotation_joint" type="continuous">
       <parent link="front_left_wheel_steering_rotation_link"/>
@@ -184,11 +193,11 @@
   </joint>
   <joint name="front_right_wheel_steering_joint" type="revolute">
-    <parent link="base_link"/>
+    <parent link="steering_link"/>
     <child link="front_right_wheel_steering_rotation_link"/>
     <origin xyz="0.2 -0.2 0.1" rpy="0 0 0"/>
     <axis xyz="0 0 1"/>
-    <limit lower="-0.5236" upper="0.5236" effort="10" velocity="1.0"/> <!-- Limite de direção (±30 graus) -->
-  </joint>
-  <!--Link intermediário para a rotação da roda dianteira esquerda-->
+    <limit lower="-0.5236" upper="0.5236" effort="10" velocity="1.0"/> <!-- (±30 degrees) -->
+  </joint>
+  <!--Link to connect the steering and rotation joints-->
   <link name="front_right_wheel_steering_rotation_link">
     <visual>
@@ -202,5 +211,4 @@
     </inertial>
   </link>
-  <!-- Junta de rotação para o eixo y (rotação da roda) -->
   <joint name="front_right_wheel_rotation_joint" type="continuous">
     <parent link="front_right_wheel_steering_rotation_link"/>
@@ -210,4 +218,15 @@
     <limit effort="100" velocity="100"/>
     <joint_properties damping="1.0" friction="1.0"/>
+  </joint>
+  <!--This two joints are the ackermann_steering_controller inputs-->
+  <joint name="steering_joint" type="fixed">
+    <parent link="base_link"/>
+    <child link="steering_link"/>
+    <origin xyz="0 0 0" rpy="0 0 0"/>
+  </joint>
+  <joint name="rear_axle_joint" type="fixed">
+    <parent link="base_link"/>
+    <child link="rear_axle_link"/>
+    <origin xyz="-0 0 0" rpy="0 0 0"/>
   </joint>
 <transmission name="front_left_wheel_steering_trans">
