Commit message: Update skid_steer_mid360.xacro
- Increase the Livox height 
- Include the ground_truth topic
- Disable the Livox point cloud visualization in Gazebo;
- Change the IMU from Gazebo plugin to Hector plugin (http://wiki.ros.org/hector_gazebo_plugins)

File: urdf/skid_steer_mid360.xacro (robot description, xacro)
@@ -176,35 +176,6 @@
     <joint_properties damping="1.0" friction="1.0"/>
   </joint>
-    <!-- IMU Sensor -->
-    <link name="imu_link">
-        <inertial>
-            <origin xyz="0 0 0" />
-            <mass value="0.01" />
-            <inertia ixx="0.0001" ixy="0" ixz="0" iyy="0.0001" iyz="0" izz="0.0001" />
-        </inertial>
-        <visual>
-            <origin xyz="0 0 0" />
-            <geometry>
-                <box size="0.01 0.01 0.01" />
-            </geometry>
-        </visual>
-    </link>
-    <joint name="imu_joint" type="fixed">
-        <parent link="base_link" />
-        <child link="imu_link" />
-        <origin xyz="0 0 0.16" rpy="0 0 0" />
-    </joint>
-    <gazebo reference="imu_link">
-        <sensor name="my_imu" type="imu">
-            <always_on>true</always_on>
-            <plugin name="my_imu_plugin" filename="libgazebo_ros_imu_sensor.so">
-                <topicName>/imu</topicName>
-                <updateRateHZ>100</updateRateHZ>
-                <frameName>imu_link</frameName>
-            </plugin>
-        </sensor>
-    </gazebo>
-    <!--Sensor LiDAR 2D -->
-    <link name="lidar_link">
+  <!-- IMU Sensor -->
+  <link name="imu_link">
       <inertial>
           <origin xyz="0 0 0" />
@@ -218,54 +189,87 @@
           </geometry>
       </visual>
-    </link>
-    <joint name="lidar_joint" type="fixed">
-        <parent link="base_link" />
-        <child link="lidar_link" />
-        <origin xyz="0 0 0.21" rpy="0 0 0" />
-    </joint>
-    <gazebo reference="lidar_link">
-      <sensor type="ray" name="laser_livox">
-        <pose>0 0 0.0 0 0 0</pose>
-        <visualize>true</visualize>
-        <always_on>True</always_on>
-        <update_rate>10</update_rate>
-        <!-- This ray plgin is only for visualization. -->
-        <plugin name="gazebo_ros_laser_controller" filename="liblivox_laser_simulation.so">
-			  <ray>
-			  <scan>
-				  <horizontal>
-				    <samples>100</samples>
-				    <resolution>1</resolution>
-				    <min_angle>-3.1415926535897931</min_angle>
-            <max_angle>3.1415926535897931</max_angle>
-				  </horizontal>
-				  <vertical>
-				    <samples>50</samples>
-				    <resolution>1</resolution>
-				    <min_angle>-3.1415926535897931</min_angle>
-            <max_angle>3.1415926535897931</max_angle>
-				  </vertical>
-			  </scan>
-			  <range>
-				  <min>0.1</min>
-				  <max>40</max>
-				  <resolution>1</resolution>
-			  </range>
-			  <noise>
-				  <type>gaussian</type>
-				  <mean>0.0</mean>
-				  <stddev>0.0</stddev>
-			  </noise>
-			  </ray>
-          <visualize>True</visualize>
-		      <samples>20000</samples>
-		      <downsample>1</downsample>
-		      <csv_file_name>mid360-real-centr.csv</csv_file_name>
-          <publish_pointcloud_type>2</publish_pointcloud_type>
-		      <ros_topic>/livox/lidar</ros_topic>
-          <frameName>base_link</frameName>
-        </plugin>
-      </sensor>
-    </gazebo>
+  </link>
+  <joint name="imu_joint" type="fixed">
+      <parent link="base_link" />
+      <child link="imu_link" />
+      <origin xyz="0 0 0.16" rpy="0 0 0" />
+  </joint>
+  <gazebo>
+    <plugin name="imu_controller" filename="libhector_gazebo_ros_imu.so">
+      <robotNamespace>/</robotNamespace>
+      <updateRate>50.0</updateRate>
+      <bodyName>base_link</bodyName>
+      <topicName>imu/data</topicName>
+      <accelDrift>0.005 0.005 0.005</accelDrift>
+      <accelGaussianNoise>0.005 0.005 0.005</accelGaussianNoise>
+      <rateDrift>0.005 0.005 0.005 </rateDrift>
+      <rateGaussianNoise>0.005 0.005 0.005 </rateGaussianNoise>
+      <headingDrift>0.005</headingDrift>
+      <headingGaussianNoise>0.005</headingGaussianNoise>
+    </plugin>
+  </gazebo>
+  <!--Sensor LiDAR 3D -->
+  <link name="lidar_link">
+    <inertial>
+        <origin xyz="0 0 0" />
+        <mass value="0.01" />
+        <inertia ixx="0.0001" ixy="0" ixz="0" iyy="0.0001" iyz="0" izz="0.0001" />
+    </inertial>
+    <visual>
+        <origin xyz="0 0 0" />
+        <geometry>
+            <box size="0.01 0.01 0.01" />
+        </geometry>
+    </visual>
+  </link>
+  <joint name="lidar_joint" type="fixed">
+      <parent link="base_link" />
+      <child link="lidar_link" />
+      <origin xyz="0 0 0.31" rpy="0 0 0" />
+  </joint>
+  <gazebo reference="lidar_link">
+    <sensor type="ray" name="laser_livox">
+      <pose>0 0 0.0 0 0 0</pose>
+      <visualize>false</visualize>
+      <always_on>True</always_on>
+      <update_rate>10</update_rate>
+      <!-- This ray plgin is only for visualization. -->
+      <plugin name="gazebo_ros_laser_controller" filename="liblivox_laser_simulation.so">
+      <ray>
+      <scan>
+        <horizontal>
+          <samples>100</samples>
+          <resolution>1</resolution>
+          <min_angle>-3.1415926535897931</min_angle>
+          <max_angle>3.1415926535897931</max_angle>
+        </horizontal>
+        <vertical>
+          <samples>50</samples>
+          <resolution>1</resolution>
+          <min_angle>-3.1415926535897931</min_angle>
+          <max_angle>3.1415926535897931</max_angle>
+        </vertical>
+      </scan>
+      <range>
+        <min>0.1</min>
+        <max>40</max>
+        <resolution>1</resolution>
+      </range>
+      <noise>
+        <type>gaussian</type>
+        <mean>0.0</mean>
+        <stddev>0.0</stddev>
+      </noise>
+      </ray>
+        <visualize>True</visualize>
+        <samples>20000</samples>
+        <downsample>1</downsample>
+        <csv_file_name>mid360-real-centr.csv</csv_file_name>
+        <publish_pointcloud_type>2</publish_pointcloud_type>
+        <ros_topic>/livox/lidar</ros_topic>
+        <frameName>base_link</frameName>
+      </plugin>
+    </sensor>
+  </gazebo>
   <!-- GPS Sensor -->
   <link name="gps_link">
@@ -323,3 +327,13 @@
     </plugin>
   </gazebo>
+  <!-- Ground truth -->
+    <gazebo>
+        <plugin name="gazebo_ros_p3d" filename="libgazebo_ros_p3d.so">
+            <alwaysOn>true</alwaysOn>
+            <updateRate>20.0</updateRate>
+            <bodyName>base_link</bodyName>
+            <topicName>ground_truth</topicName>
+            <robotNamespace>/</robotNamespace>
+        </plugin>
+    </gazebo>
 </robot>
